File: pcb/TashRecorder.kicad_sch (KiCad schematic)
At the start: 49 parts, among them J1 RCJ-013, J2 Mini-DIN-8, J3 Conn_01x04, SW1 EG 1224 SPDT, U1 LM385Z-2.5, U2 LM385Z-2.5, U3 OPA2337, U4 PIC12F1501-xP

Commit message: cleaned BOM
Parts:
- H1, H2, H3, H4, J3: now left out of the parts list
- R14, R15: value 47 -> 47Ω
- R7: value 220k -> 220kΩ
Changed lines of the file:
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@@
 			)
 		)
-		(property "Value" "47"
+		(property "Value" "47Ω"
 			(at 247.65 124.0536 90)
 			(effects
@@
 			)
 		)
-		(property "Value" "47"
+		(property "Value" "47Ω"
 			(at 247.65 73.2536 90)
 			(effects
@@
 		(unit 1)
 		(exclude_from_sim no)
-		(in_bom yes)
+		(in_bom no)
 		(on_board yes)
 		(dnp no)
@@
 		(unit 1)
 		(exclude_from_sim no)
-		(in_bom yes)
+		(in_bom no)
 		(on_board yes)
 		(dnp no)
@@
 		(unit 1)
 		(exclude_from_sim no)
-		(in_bom yes)
+		(in_bom no)
 		(on_board yes)
 		(dnp no)
@@
 		(unit 1)
 		(exclude_from_sim no)
-		(in_bom yes)
+		(in_bom no)
 		(on_board yes)
 		(dnp no)
@@
 			)
 		)
-		(property "Value" "220k"
+		(property "Value" "220kΩ"
 			(at 114.3 124.0536 90)
 			(effects
@@
 		(unit 1)
 		(exclude_from_sim no)
-		(in_bom yes)
-		(on_board yes)
-		(dnp no)
+		(in_bom no)
+		(on_board yes)
+		(dnp no)
